File: pcb/PRAHARI.kicad_pcb (KiCad board)
At the start: 2 copper layers, 70 x 40 mm, 38 parts, among them J1 MAX30102, J2 MAX30208, J3 AHT20, J4 LiPo 3.7V 350mAh, J5 HAPTIC, J6 ANT WHIP, J7 OLED 0.91in, Q1 2N7002, U1 XIAO nRF52840 Sense, U2 Ra-01SH SX1262, U3 ATECC608A-SSHDA, U4 DW01A, U5 FS8205A

Commit message: Add prototype-evolution section (three-question format) to PDF report
Parts:
- removed C7: 100nF, Capacitor_SMD:C_0805_2012Metric
- removed R6: 100R, Resistor_SMD:R_0805_2012Metric
- removed U4: DW01A, Package_TO_SOT_SMD:SOT-23-6
- removed U5: FS8205A, Package_TO_SOT_SMD:SOT-23-6
- J1: value MAX30102 -> MAX30100
- J2: value MAX30208 -> MLX90614
- J4: value LiPo 3.7V 350mAh -> LiPo 3.7V
- J7: value OLED 0.91in -> OLED 0.96in
- U2: value Ra-01SH SX1262 -> Ra-02 SX1278; footprint PRAHARI:Ai-Thinker_Ra-01SH -> PRAHARI:Ai-Thinker_Ra-02
- moved C1 23.8 mm to (61.0, 42.0), turned to 0 degrees
- moved C3 19.7 mm to (55.0, 42.0), turned to 0 degrees
- moved J6 3.16 mm to (45.0, 42.0), turned to 90 degrees
- moved U2 1.50 mm to (50.0, 53.5)
Connections:
- J4 pad 2: BAT_NEG -> GND
- U1 pad 2: LORA_BUSY -> LORA_DIO0
- U2 pad 1: ANT -> GND
- U2 pad 10: LORA_TXEN -> SPI_MOSI
- U2 pad 11: LORA_RXEN -> SPI_SCK
- U2 pad 12: SPI_SCK -> GND
- U2 pad 13: SPI_MISO -> +3V3
- U2 pad 14: SPI_MOSI -> LORA_RST
- U2 pad 15: LORA_NSS -> ANT
- U2 pad 2: GND -> LORA_DIO5
- U2 pad 3: +3V3 -> LORA_DIO4
- U2 pad 4: LORA_RST -> LORA_DIO3
- U2 pad 5: LORA_BUSY -> LORA_DIO2
- U2 pad 7: LORA_DIO2 -> LORA_DIO0
- U2 pad 8: LORA_DIO3 -> LORA_NSS
- U2 pad 9: GND -> SPI_MISO
Routing:
- net LORA_BUSY: track 48.0 -> 0.00 mm, vias 3 -> 0
- net SCL: track 116.6 -> 76.5 mm, vias 8 -> 2
- net LORA_DIO1: track 0.00 -> 38.5 mm, vias 0 -> 1
- net LORA_DIO0: track 0.00 -> 25.9 mm, vias 0 -> 2
- net LORA_RST: track 53.5 -> 29.6 mm
- net BAT_NEG: track 12.9 -> 0.00 mm
- net DW_OD: track 11.2 -> 0.00 mm
- net PPG_INT: track 60.8 -> 51.3 mm, vias 0 -> 1
- net DW_OC: track 7.27 -> 0.00 mm, vias 2 -> 0
- net SPI_SCK: track 50.7 -> 55.2 mm, vias 3 -> 1
- net SDA: track 71.8 -> 67.7 mm, vias 4 -> 3
- net +3V3: track 132.8 -> 136.8 mm
- net LORA_NSS: track 19.7 -> 23.1 mm, vias 0 -> 1
- net ANT: track 5.69 -> 2.30 mm
- net SPI_MISO: track 40.8 -> 38.5 mm
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Other:
- board text added: "PRAHARI rev A"
- board text added: "rev A - 70 x 40 mm - 2 layer"
- board text removed: "PRAHARI rev B"
- board text removed: "rev B - 70 x 40 mm - 2 layer - 868 MHz"
