File: pcb/PRAHARI.kicad_sch (KiCad schematic)
At the start: 38 parts, among them J1 MAX30102, J2 MAX30208, J3 AHT20, J4 LiPo 3.7V 350mAh, J5 HAPTIC, J6 ANT WHIP, J7 OLED 0.91in, Q1 2N7002, U1 XIAO nRF52840 Sense, U2 Ra-01SH SX1262, U3 ATECC608A-SSHDA, U4 DW01A, U5 FS8205A

Commit message: Add prototype-evolution section (three-question format) to PDF report
Parts:
- removed C7: 100nF, Capacitor_SMD:C_0805_2012Metric, symbol Device:C
- removed R6: 100R, Resistor_SMD:R_0805_2012Metric, symbol Device:R
- removed U2: Ra-01SH SX1262, PRAHARI:Ai-Thinker_Ra-01SH, symbol PRAHARI:Ai-Thinker_Ra-01SH
- removed U4: DW01A, Package_TO_SOT_SMD:SOT-23-6, symbol PRAHARI:DW01A
- removed U5: FS8205A, Package_TO_SOT_SMD:SOT-23-6, symbol PRAHARI:FS8205A
- added U2: Ra-02 SX1278, PRAHARI:Ai-Thinker_Ra-02, symbol PRAHARI:Ai-Thinker_Ra-02
- J1: value MAX30102 -> MAX30100
- J2: value MAX30208 -> MLX90614
- J4: value LiPo 3.7V 350mAh -> LiPo 3.7V
- J7: value OLED 0.91in -> OLED 0.96in
Connections:
- net BAT_NEG is gone; now on net GND: J4.2 (Pin_2)
- net +3V3: now also U2.13 (3V3)
- net GND: now also U2.1 (GND), U2.12 (GND), U2.16 (GND)
- net LORA_DIO1: now also U2.6 (DIO1)
- net LORA_DIO2: now also U2.5 (DIO2)
- net LORA_DIO3: now also U2.4 (DIO3)
- net LORA_NSS: now also U2.8 (NSS)
- net LORA_RST: now also U2.14 (RST)
- net SPI_MISO: now also U2.9 (MISO)
- net SPI_MOSI: now also U2.10 (MOSI)
- net SPI_SCK: now also U2.11 (SCK)
- net at J6.1 (Pin_1): now also U2.15 (ANT)
- net LORA_BUSY renamed LORA_DIO0
- net LORA_DIO0: now also U2.7 (DIO0)
- new net LORA_DIO4: U2.3 (DIO4)
- new net LORA_DIO5: U2.2 (DIO5)
- no-connect marks 5 -> 4
Other:
- note added: "LoRa 433 MHz (SX1278)"
- note added: "POWER"
- note removed: "LoRa 868 MHz (SX1262)"
- note removed: "POWER + BATTERY PROTECTION"
